File: Eagle/Cargador 12,6V-5A.sch (EAGLE design)
At the start: 13 parts

Commit message: Terminado etapa integrado OB2269
Parts:
- added C2: 100n, rcl:C-US050-024X044
- added C5: 1u, rcl:C-US050-024X044
- added C6: 22uf, rcl:CPOL-USE5-10.5
- added D1, D2, D3: MBR0520LT, diode:MBR0520LT
- added EC1: 150u/400v, rcl:CPOL-USE5-10.5
- added IC1: OB2269, Circuitos-Creativos-Integrados-8pin:OB2269
- added L3: (no value), trafo-siemens:ST-D4
- added Q1: IRF840, transistor-fet:IRF840
- added R0.1: 0R, rcl:R-US_0204/7
- added R10: 200, rcl:R-US_0204/7
- added R3A, R3A1: 560k, rcl:R-US_0204/7
- added R4: 56k, rcl:R-US_0204/7
- added R5: 100, rcl:R-US_0204/7
- added R8, R9: 24k, rcl:R-US_0204/7
- C4: value 150u/400v -> 33n; device rcl:CPOL-USE5-10.5 -> rcl:C-US050-024X044
Connections:
- new net N$10: C5.1, IC1.FB
- new net N$11: IC1.VDD, R0.1.1
- new net N$12: C6.+, D3.C, R0.1.2
- new net N$13: D3.A, R10.1
- new net N$14: L3.3E, R10.2
- new net N$15: IC1.RI, R8.2
- new net N$16: IC1.RT, R9.2
- new net N$17: C4.1, IC1.SENSE, Q1.S
- new net N$18: D2.C, IC1.GATE, R5.1
- new net N$19: L3.1A, R4.1
- new net N$20: D2.A, Q1.G, R5.2
- new net N$21: D1.A, L3.1E, Q1.D
- new net N$22: D1.C, R4.2
- new net N$7: R3A.2, R3A1.1
- new net N$9: C2.1, IC1.VIN, R3A1.2
- net AGND: now also C2.2, C4.2, C5.2, C6.-, EC1.-, IC1.GND, L3.3A, R8.1, R9.1; no longer C4.-
- net N$8: now also EC1.+, R3A.1; no longer C4.+
